File: kicad/gonogo-light/timer-light.sch (KiCad schematic (older format))
At the start: 58 parts, among them J1 Screw_Terminal_01x02, J2 Screw_Terminal_01x04, K1 FINDER-30.22, Q1 2N2222, Q2 2N2222, SW1 SW_DIP_x04, SW2 SW_DIP_x08, SW3 SW_DIP_x04, SW4 SW_DIP_x08, U1 4011, U10 4011, U11 4040, U12 4012, U13 4068, U2 4040, U3 4060, U4 4012, U5 4013, U6 4011, U7 4040, U8 4068, U9 4012, Y1 32,768 kHz

Commit message: correction des erreurs et ajout de capas de reset sur poweron
Parts:
- added C20: 100nF, Capacitor_THT:C_Rect_L7.2mm_W2.5mm_P5.00mm_FKS2_FKP2_MKS2_MKP2, symbol timer-light-rescue:C-Device
- 2A1, 2A2: symbol Device:Fuse_Small -> timer-light-rescue:Fuse_Small-Device
- C1, C10, C11, C12, C13, C14, C15, C16, C17, C18, C2, C3, C4, C5, C6, C7, C8, C9: symbol Device:C -> timer-light-rescue:C-Device
- C19: symbol Device:CP -> timer-light-rescue:CP-Device
- D1: symbol Device:D_Small -> timer-light-rescue:D_Small-Device
- D2: symbol Device:LED -> timer-light-rescue:LED-Device
- D3: symbol Diode:1N4001 -> timer-light-rescue:1N4001-Diode
- F1: symbol Device:Polyfuse_Small -> timer-light-rescue:Polyfuse_Small-Device
- J1: symbol Connector:Screw_Terminal_01x02 -> timer-light-rescue:Screw_Terminal_01x02-Connector
- J2: symbol Connector:Screw_Terminal_01x04 -> timer-light-rescue:Screw_Terminal_01x04-Connector
- JP1, JP2: symbol Device:Jumper_NC_Dual -> timer-light-rescue:Jumper_NC_Dual-Device
- K1: symbol Relay:FINDER-30.22 -> timer-light-rescue:FINDER-30.22-Relay
- Q1, Q2: symbol Transistor_BJT:BC107 -> timer-light-rescue:BC107-Transistor_BJT
- R1, R2, R3: symbol Device:R -> timer-light-rescue:R-Device
- R4: value 10k -> Voir Note 1; symbol Device:R -> timer-light-rescue:R-Device
- RN1, RN3: symbol Device:R_Network04 -> timer-light-rescue:R_Network04-Device
- RN2, RN4: symbol Device:R_Network08 -> timer-light-rescue:R_Network08-Device
- SW1, SW3: symbol Switch:SW_DIP_x04 -> timer-light-rescue:SW_DIP_x04-Switch
- SW2, SW4: symbol Switch:SW_DIP_x08 -> timer-light-rescue:SW_DIP_x08-Switch
- U1, U10, U6: symbol 4xxx:4011 -> timer-light-rescue:4011-4xxx
- U11, U2, U7: symbol 4xxx:4040 -> timer-light-rescue:4040-4xxx
- U12, U4, U9: symbol 4xxx:4012 -> timer-light-rescue:4012-4xxx
- U13, U8: symbol 4xxx_IEEE:4068 -> timer-light-rescue:4068-4xxx_IEEE
- U5: symbol 4xxx:4013 -> timer-light-rescue:4013-4xxx
- Y1: symbol Device:Crystal -> timer-light-rescue:Crystal-Device
Connections:
- wire segments 374 -> 378
Other:
- note added: "Note 1 :\nR4 = 330 ohms sous 5V\nR4 = 1 Kohms sous 12V"
- moved on the sheet: U6A, U6B
